File: db37kx.kicad_pcb (KiCad board)
At the start: 2 copper layers, 70.5 x 31.7 mm, 12 parts, among them J1 1989748, J2 54-00299, J3 54-00299, J4 54-00176, J5 54-00299, J6 54-00299, J7 54-00299, J8 5747847-6

Commit message: rev B start
Parts:
- removed H1, H2, H3, H4: MountingHole_Pad, MountingHole:MountingHole_3.2mm_M3_DIN965_Pad_TopBottom
- added S1: 9774030360R, Spacer_Wuerth:9774030360R, F.Cu at (109.0, 90.0)
- J8: value 5747847-6 -> K85X-CD-37S; footprint Connector_Dsub_TE:CONN_5747847-6_TYC -> Connector_Dsub_Kycon:K85X-CD-37S
- moved J1 84.7 mm to (40.6, 35.8)
- moved J5 73.9 mm to (79.0, 80.0), turned to -90 degrees
- moved J6 68.2 mm to (94.0, 80.0), turned to -90 degrees
- moved J8 63.2 mm to (124.0, 115.6), turned to 180 degrees
- moved J2 55.0 mm to (169.0, 80.0), turned to -90 degrees
- moved J3 31.5 mm to (154.0, 80.0), turned to -90 degrees
- moved J4 21.7 mm to (124.0, 80.0), turned to -90 degrees
- moved J7 12.0 mm to (139.0, 80.0), turned to -90 degrees
Routing:
- net /RADIO AF OUT GND: track 37.0 -> 0.00 mm
- net /RADIO MIC IN GND: track 31.7 -> 0.00 mm
- net /PTT: track 31.0 -> 0.00 mm
- net /RADIO AF OUT: track 30.7 -> 0.00 mm
- net /RADIO MIC IN: track 27.3 -> 0.00 mm
- net /FILTER IN: track 26.5 -> 0.00 mm
- net /RS232 OUT: track 26.4 -> 0.00 mm
- net /CW OUT: track 26.0 -> 0.00 mm
- net /FSW IN: track 24.1 -> 0.00 mm
- net /MIC: track 13.6 -> 0.00 mm
- net /RADIO_R_PASSTHRU: track 9.25 -> 0.00 mm
- net /MIC GND: track 8.10 -> 0.00 mm
- net +12V: track 7.17 -> 0.10 mm
- net /RS232CTS: track 3.42 -> 0.00 mm
- net /RS-TTL OUT: track 2.77 -> 0.00 mm
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- removed copper zone on B.Cu, net GND
- removed copper zone on F.Cu, net GND
Other:
- board size 70.5 x 31.7 mm -> 102 x 48 mm
- board text added: "Connector outline"
- board text added: "GND"
- board text added: "board guide"
