File: db37kx.kicad_sch (KiCad schematic)
At the start: 12 parts, among them J1 1989748, J2 54-00299, J3 54-00299, J4 54-00176, J5 54-00299, J6 54-00299, J7 54-00299, J8 5747847-6

Commit message: rev B start
Parts:
- removed H1, H2, H3, H4: MountingHole_Pad, MountingHole:MountingHole_3.2mm_M3_DIN965_Pad_TopBottom, symbol Mechanical:MountingHole_Pad
- added S1: 9774030360R, Spacer_Wuerth:9774030360R, symbol Spacer_Wuerth:9774030360R
- J8: value 5747847-6 -> K85X-CD-37S; footprint Connector_Dsub_TE:CONN_5747847-6_TYC -> Connector_Dsub_Kycon:K85X-CD-37S; symbol Connector_Dsub_TE:5747847-6 -> Connector_Dsub_Kycon:K85X-CD-37S; DPN A32130-ND -> (none); Digi-KeyPN (none) -> 2092-K85X-CD-37S-ND; MPN 5747847-6 -> K85X-CD-37S; Manufacturer TE -> Kycon; MouserPN (none) -> 806-K85X-CD-37S
Connections:
- net GND: now also S1.1 (Pin_1)
